Commit message: Added Robotiq 2f 140 gripper to robot arm

File: robot_model/mpo_700/mpo_700.urdf.xacro (robot description, xacro)
@@ -392,4 +392,19 @@
       <origin xyz="0.133 0.0 0.416" rpy="0.0 0.0 -1.5708" />
     </xacro:ur_robot>
+    <xacro:unless value="${gripper == ''}">
+      <!-- ur_adapter for gripper-->
+      <xacro:include filename="$(find robotiq_description)/urdf/ur_to_robotiq_adapter.urdf.xacro"/>
+      <xacro:ur_to_robotiq
+          prefix=""
+          parent="$(arg tf_prefix)tool0"
+          child="neo_gripper_mount_link"
+          rotation="${pi/2}"
+          />
+      <!-- add gripper-->
+      <xacro:include filename="$(find robotiq_description)/urdf/robotiq_2f_140_macro.urdf.xacro"/>
+      <xacro:robotiq_gripper name="robotiq_gripper" prefix="" parent="neo_gripper_mount_link" include_ros2_control="true" sim_ignition="true">
+          <origin xyz="0 0 0" rpy="0 0 -${pi / 2}"/>
+      </xacro:robotiq_gripper>
+    </xacro:unless>
   </xacro:unless>
 </robot>

Commit message: adding gripper to the URDF and dependency update

File: robot_model/mpo_700/mpo_700.urdf.xacro (robot description, xacro)
@@ -5,7 +5,9 @@
   <xacro:arg name="use_imu" default="false"/>
   <xacro:arg name="use_d435" default="false"/>
+  <xacro:arg name="gripper_type" default=""/>
   <xacro:property name="arm" value="$(arg arm_type)"/>
   <xacro:property name="imu" value="$(arg use_imu)"/>
   <xacro:property name="d435" value="$(arg use_d435)"/>
+  <xacro:property name="gripper" value="$(arg gripper_type)"/>
   <!-- When there is an arm mounted, the joints of the wheels needs
   to be of fixed type. The reason being, both the drive modules and
@@ -403,5 +405,5 @@
       <!-- add gripper-->
       <xacro:include filename="$(find robotiq_description)/urdf/robotiq_2f_140_macro.urdf.xacro"/>
-      <xacro:robotiq_gripper name="robotiq_gripper" prefix="" parent="neo_gripper_mount_link" include_ros2_control="true" sim_ignition="true">
+      <xacro:robotiq_gripper name="robotiq_gripper" prefix="" parent="neo_gripper_mount_link" include_ros2_control="true">
           <origin xyz="0 0 0" rpy="0 0 -${pi / 2}"/>
       </xacro:robotiq_gripper>
